File: PCB_rev_B3/Replicape_B3.brd (EAGLE design)
At the start: 107.3 x 69.5 mm, 244 parts, among them IC1 TMC2100-LA, IC10 74AHC1G126DCK, IC11 74AHC1G126DCK, IC12 TMC2100-LA, IC13 74AHC1G126DCK, IC14 74AHC1G126DCK, IC15 TMC2100-LA, IC16 74AHC1G126DCK, IC17 74AHC1G126DCK, IC18 74AHC1G126DCK, IC19 74AHC1G126DCK, IC2 TMC2100-LA, IC3 74AHC1G126DCK, IC4 74AHC1G126DCK, IC5 TMC2100-LA, IC6 74AHC1G126DCK, IC7 74AHC1G126DCK, IC8 74AHC1G126DCK, IC9 74AHC1G126DCK, P8 F-2X23-, P9 F-2X23-, Q1 AON6758, Q2 AON6758, Q3 AON6758, U1 SN74AHC595PW, U10 RT8268, U11 PCA9685PW, U18 CAT24C256, U19 CD4050BD, U2 SN74AHC595PW, U3 SN74AHC595PW, U4 SN74AHC595PW, U5 SN74AHC595PW, U6 RT8268, X1 22-05-7038-03, X10 22-05-7038-03, X11 22-05-7028-02, X12 22-05-7048-04, X13 22-05-7038-03, X14 22-05-7048-04, X15 22-05-7048-04, X16 22-05-7048-04, X17 22-05-7048-04, X18 22-05-7048-04, X19 22-05-7038-03, X2 MSTBA4, X20 MSTBA4, X21 MSTBA2, X22 22-05-7038-03, X23 22-05-7038-03, X3 MSTBA2, X4 22-05-7028-02, X5 22-05-7028-02, X6 22-05-7028-02, X7 22-05-7028-02, X8 22-05-7028-02, X9 22-05-7028-02

Commit message: Updated readmen
Changed lines of the file:
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@@
 <layer number="23" name="tOrigins" color="15" fill="1" visible="yes" active="yes"/>
 <layer number="24" name="bOrigins" color="15" fill="1" visible="yes" active="yes"/>
-<layer number="25" name="tNames" color="7" fill="1" visible="no" active="yes"/>
-<layer number="26" name="bNames" color="7" fill="1" visible="no" active="yes"/>
+<layer number="25" name="tNames" color="7" fill="1" visible="yes" active="yes"/>
+<layer number="26" name="bNames" color="7" fill="1" visible="yes" active="yes"/>
 <layer number="27" name="tValues" color="7" fill="1" visible="no" active="yes"/>
 <layer number="28" name="bValues" color="7" fill="1" visible="no" active="yes"/>
@@
 </element>
 <element name="U18" library="custom" package="SOIC127P600X175-8N" value="CAT24C256" x="33.575" y="51" smashed="yes" rot="R270">
-<attribute name="NAME" x="30.7996" y="51.7638" size="0.6096" layer="25" ratio="10" rot="SR90"/>
+<attribute name="NAME" x="30.22" y="54.0544" size="0.6096" layer="25" ratio="10" rot="SR270"/>
+<attribute name="VALUE" x="27.86" y="54.4544" size="2.0828" layer="27" ratio="10" rot="SR270"/>
 </element>
 <element name="LOGO1" library="ohw-logo" package="OSHW_FILLX200_NOTEXT" value="OSHW_LOGO_FILLX0200-NT" x="83.8584" y="17.5102" smashed="yes"/>
