File: Reach_rev_B0/Reach_B0.sch (EAGLE design)
At the start: 91 parts, among them IC1 TMC2100-LA, IC18 74AHC1G126DCK, IC2 TMC2100-LA, IC3 74AHC1G126DCK, IC4 74AHC1G126DCK, IC8 74AHC1G126DCK, IC9 74AHC1G126DCK, P8 F-2X23-, P9 F-2X23-, Q2 AON6758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

Commit message: Added new version eeprom data
Connections:
- new net THERMO_1: P9.37
- new net THERMO_2: P9.38
Changed lines of the file:
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@@
+</segment>
+</net>
+<net name="THERMO_1" class="0">
+<segment>
+<pinref part="P9" gate="G$1" pin="37"/>
+<wire x1="563.88" y1="43.18" x2="538.48" y2="43.18" width="0.1524" layer="91"/>
+<label x="538.48" y="43.18" size="1.778" layer="95"/>
+</segment>
+</net>
+<net name="THERMO_2" class="0">
+<segment>
+<pinref part="P9" gate="G$1" pin="38"/>
+<wire x1="579.12" y1="43.18" x2="604.52" y2="43.18" width="0.1524" layer="91"/>
+<label x="581.66" y="43.18" size="1.778" layer="95"/>
 </segment>
 </net>

Commit message: Added a Collada (DAE) file
Parts:
- added IC5: 74AHC1G126DCK, 74xx-little-de:74AHC1G126DCK
- added J1: 22-05-7038-03, con-molex:22-05-7038-03
- added U3: TS3A5018PW, Texas Instruments_By_element14_Batch_1:TS3A5018PW
Connections:
- removed net ENABLE_XYZ: IC1.DRV_ENN_CFG6, IC18A.O, IC2.DRV_ENN_CFG6
- removed net SERVO_0_EN: U2.QA
- new net ENABLE_A: IC1.DRV_ENN_CFG6, IC18A.O
- new net ENABLE_B: IC2.DRV_ENN_CFG6, IC5A.O
- new net N$1: IC5A.I, U2.QA
- new net N$11: C26.2, X8-1.S
- new net N$9: C46.2
- net GND: no longer C26.2, C46.2, X8-1.S
- net N$240: no longer R18.1, R40.1
- net VDD_ADC: no longer R18.2
Other:
- moved on the sheet: C26, C46, R13, R18, R24, R38, R40, X8-1, X8-2
